File: Hardware/Hardware.kicad_pcb (KiCad board)
At the start: 2 copper layers, 108 x 61.2 mm, 66 parts, among them J1 LINEIN, J2 MICIN, J3 Raspberry_Pi_2_3, J4 LOUT, J5 HPOUT, SW1 JS5208, U1 MCP3004, U2 WM8731SEDS, Y1 CO4305-12.000

Commit message: Re-made renders of PCB.
Parts:
- added G***: LOGO, signl:signl_logo, B.Cu at (165.1, 54.6)
